Commit message: chore: relocate project to D:\g1_guide with its own CLAUDE.md
Co-Authored-By: Claude Opus 5.5 <noreply@anthropic.com>

File: ws/src/g1_guide/urdf/g1_glide.urdf (robot description, URDF)
Before this commit: robot g1_29dof_mode_11, 41 links, 40 joints
Links:
- link head_link: geometry collision mesh filename=/mnt/d/g1_guide/ws/src/g1_description/meshes/head_link.STL; visual mesh filename=/mnt/d/g1_guide/ws/src/g1_description/meshes/head_link.STL
- link left_ankle_pitch_link: geometry collision mesh filename=/mnt/d/g1_guide/ws/src/g1_description/meshes/left_ankle_pit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; visual mesh filename=/mnt/d/g1_guide/ws/src/g1_description/meshes/left_ankle_pit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
- link left_ankle_roll_link: geometry collision sphere radius=0.005; collision sphere radius=0.005
- link left_elbow_link: geometry collision mesh filename=/mnt/d/g1_guide/ws/src/g1_description/meshes/left_elbow_lin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; visual mesh filename=/mnt/d/g1_guide/ws/src/g1_description/meshes/left_elbow_lin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
- link left_hip_pitch_link: geometry collision mesh filename=/mnt/d/g1_guide/ws/src/g1_description/meshes/left_hip_pitch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; visual mesh filename=/mnt/d/g1_guide/ws/src/g1_description/meshes/left_hip_pitch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
- link left_hip_roll_link: geometry collision mesh filename=/mnt/d/g1_guide/ws/src/g1_description/meshes/left_hip_roll_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; visual mesh filename=/mnt/d/g1_guide/ws/src/g1_description/meshes/left_hip_roll_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
- link left_hip_yaw_link: geometry collision mesh filename=/mnt/d/g1_guide/ws/src/g1_description/meshes/left_hip_yaw_l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; visual mesh filename=/mnt/d/g1_guide/ws/src/g1_description/meshes/left_hip_yaw_l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
- link left_knee_link: geometry collision mesh filename=/mnt/d/g1_guide/ws/src/g1_description/meshes/left_knee_link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; visual mesh filename=/mnt/d/g1_guide/ws/src/g1_description/meshes/left_knee_link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
- link left_rubber_hand: geometry visual mesh filename=/mnt/d/g1_guide/ws/src/g1_description/meshes/left_rubber_ha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
- link left_shoulder_pitch_link: geometry collision cylinder length=0.05 radius=0.03; visual mesh filename=/mnt/d/g1_guide/ws/src/g1_description/meshes/left_shoulder_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
- link left_shoulder_roll_link: geometry collision cylinder length=0.03 radius=0.03; visual mesh filename=/mnt/d/g1_guide/ws/src/g1_description/meshes/left_shoulder_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
- link left_shoulder_yaw_link: geometry collision mesh filename=/mnt/d/g1_guide/ws/src/g1_description/meshes/left_shoulder_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; visual mesh filename=/mnt/d/g1_guide/ws/src/g1_description/meshes/left_shoulder_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
- link left_wrist_pitch_link: geometry collision mesh filename=/mnt/d/g1_guide/ws/src/g1_description/meshes/left_wrist_pit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; visual mesh filename=/mnt/d/g1_guide/ws/src/g1_description/meshes/left_wrist_pit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
- link left_wrist_roll_link: geometry collision mesh filename=/mnt/d/g1_guide/ws/src/g1_description/meshes/left_wrist_rol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; visual mesh filename=/mnt/d/g1_guide/ws/src/g1_description/meshes/left_wrist_rol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
- link left_wrist_yaw_link: geometry collision mesh filename=/mnt/d/g1_guide/ws/src/g1_description/meshes/left_wrist_yaw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; visual mesh filename=/mnt/d/g1_guide/ws/src/g1_description/meshes/left_wrist_yaw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
- link logo_link: geometry collision mesh filename=/mnt/d/g1_guide/ws/src/g1_description/meshes/logo_link.STL; visual mesh filename=/mnt/d/g1_guide/ws/src/g1_description/meshes/logo_link.STL
- link pelvis: geometry visual mesh filename=/mnt/d/g1_guide/ws/src/g1_description/meshes/pelvis_ver0529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
- link right_ankle_pitch_link: geometry collision mesh filename=/mnt/d/g1_guide/ws/src/g1_description/meshes/right_ankle_pi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; visual mesh filename=/mnt/d/g1_guide/ws/src/g1_description/meshes/right_ankle_pi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
- link right_ankle_roll_link: geometry collision sphere radius=0.005; collision sphere radius=0.005
- link right_elbow_link: geometry collision mesh filename=/mnt/d/g1_guide/ws/src/g1_description/meshes/right_elbow_li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; visual mesh filename=/mnt/d/g1_guide/ws/src/g1_description/meshes/right_elbow_li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
- link right_hip_pitch_link: geometry collision mesh filename=/mnt/d/g1_guide/ws/src/g1_description/meshes/right_hip_pitc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; visual mesh filename=/mnt/d/g1_guide/ws/src/g1_description/meshes/right_hip_pitc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
- link right_hip_roll_link: geometry collision mesh filename=/mnt/d/g1_guide/ws/src/g1_description/meshes/right_hip_roll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; visual mesh filename=/mnt/d/g1_guide/ws/src/g1_description/meshes/right_hip_roll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
- link right_hip_yaw_link: geometry collision mesh filename=/mnt/d/g1_guide/ws/src/g1_description/meshes/right_hip_yaw_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; visual mesh filename=/mnt/d/g1_guide/ws/src/g1_description/meshes/right_hip_yaw_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
- link right_knee_link: geometry collision mesh filename=/mnt/d/g1_guide/ws/src/g1_description/meshes/right_knee_lin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; visual mesh filename=/mnt/d/g1_guide/ws/src/g1_description/meshes/right_knee_lin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
- link right_rubber_hand: geometry visual mesh filename=/mnt/d/g1_guide/ws/src/g1_description/meshes/right_rubber_h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
- link right_shoulder_pitch_link: geometry collision cylinder length=0.05 radius=0.03; visual mesh filename=/mnt/d/g1_guide/ws/src/g1_description/meshes/right_shoulder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
- link right_shoulder_roll_link: geometry collision cylinder length=0.03 radius=0.03; visual mesh filename=/mnt/d/g1_guide/ws/src/g1_description/meshes/right_shoulder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
- link right_shoulder_yaw_link: geometry collision mesh filename=/mnt/d/g1_guide/ws/src/g1_description/meshes/right_shoulder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; visual mesh filename=/mnt/d/g1_guide/ws/src/g1_description/meshes/right_shoulder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
- link right_wrist_pitch_link: geometry collision mesh filename=/mnt/d/g1_guide/ws/src/g1_description/meshes/right_wrist_pi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; visual mesh filename=/mnt/d/g1_guide/ws/src/g1_description/meshes/right_wrist_pi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
- link right_wrist_roll_link: geometry collision mesh filename=/mnt/d/g1_guide/ws/src/g1_description/meshes/right_wrist_ro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; visual mesh filename=/mnt/d/g1_guide/ws/src/g1_description/meshes/right_wrist_ro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
- link right_wrist_yaw_link: geometry collision mesh filename=/mnt/d/g1_guide/ws/src/g1_description/meshes/right_wrist_ya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; visual mesh filename=/mnt/d/g1_guide/ws/src/g1_description/meshes/right_wrist_ya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
- link torso_link: geometry collision mesh filename=/mnt/d/g1_guide/ws/src/g1_description/meshes/torso_link_rev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; visual mesh filename=/mnt/d/g1_guide/ws/src/g1_description/meshes/torso_link_rev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
- link waist_roll_link: geometry visual mesh filename=/mnt/d/g1_guide/ws/src/g1_description/meshes/waist_roll_lin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
- link waist_yaw_link: geometry visual mesh filename=/mnt/d/g1_guide/ws/src/g1_description/meshes/waist_yaw_link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

Commit message: 讲解手势：展馆平移模型放开手臂，gesture_player 播放 7 个关键帧动作（M2.3）
- make_glide_urdf.py：只放开左右臂 14 个关节，手臂连杆关闭重力，
  每个关节配 gz JointPositionController（速度指令模式），并发布 /joint_states
- config/gestures.yaml：home/wave/point/present/explain_loop/emphasize/invite，
  角度按左臂约定写，右臂自动镜像
- gestures.py：关键帧插值、随机扰动、循环与插入后恢复
- arm_kinematics.py：numpy 正运动学 + 指向 IK
- gesture_player：订阅 /guide/gesture；行走中手臂锁 home，到站自动指向展品
- 用户目视验收通过

Co-Authored-By: Claude Opus 5.5 <noreply@anthropic.com>

File: ws/src/g1_guide/urdf/g1_glide.urdf (robot description, URDF)
Before this commit: robot g1_29dof_mode_11, 41 links, 40 joints
Joints:
- joint left_elbow_joint: axis (none) -> 0 1 0; limit (none) -> lower=-1.0472 upper=2.0944 effort=25 velocity=37; type fixed -> revolute
- joint left_shoulder_pitch_joint: axis (none) -> 0 1 0; limit (none) -> lower=-3.0892 upper=2.6704 effort=25 velocity=37; type fixed -> revolute
- joint left_shoulder_roll_joint: axis (none) -> 1 0 0; limit (none) -> lower=-1.5882 upper=2.2515 effort=25 velocity=37; type fixed -> revolute
- joint left_shoulder_yaw_joint: axis (none) -> 0 0 1; limit (none) -> lower=-2.618 upper=2.618 effort=25 velocity=37; type fixed -> revolute
- joint left_wrist_pitch_joint: axis (none) -> 0 1 0; limit (none) -> lower=-1.614429558 upper=1.614429558 effort=5 velocity=22; type fixed -> revolute
- joint left_wrist_roll_joint: axis (none) -> 1 0 0; limit (none) -> lower=-1.972222054 upper=1.972222054 effort=25 velocity=37; type fixed -> revolute
- joint left_wrist_yaw_joint: axis (none) -> 0 0 1; limit (none) -> lower=-1.614429558 upper=1.614429558 effort=5 velocity=22; type fixed -> revolute
- joint right_elbow_joint: axis (none) -> 0 1 0; limit (none) -> lower=-1.0472 upper=2.0944 effort=25 velocity=37; type fixed -> revolute
- joint right_shoulder_pitch_joint: axis (none) -> 0 1 0; limit (none) -> lower=-3.0892 upper=2.6704 effort=25 velocity=37; type fixed -> revolute
- joint right_shoulder_roll_joint: axis (none) -> 1 0 0; limit (none) -> lower=-2.2515 upper=1.5882 effort=25 velocity=37; type fixed -> revolute
- joint right_shoulder_yaw_joint: axis (none) -> 0 0 1; limit (none) -> lower=-2.618 upper=2.618 effort=25 velocity=37; type fixed -> revolute
- joint right_wrist_pitch_joint: axis (none) -> 0 1 0; limit (none) -> lower=-1.614429558 upper=1.614429558 effort=5 velocity=22; type fixed -> revolute
- joint right_wrist_roll_joint: axis (none) -> 1 0 0; limit (none) -> lower=-1.972222054 upper=1.972222054 effort=25 velocity=37; type fixed -> revolute
- joint right_wrist_yaw_joint: axis (none) -> 0 0 1; limit (none) -> lower=-1.614429558 upper=1.614429558 effort=5 velocity=22; type fixed -> revolute

Commit message: 视觉与人群感知：雷达数人、面向观众讲解、前置相机视觉唤醒和手势
- M5.2 雷达人群感知：people_core + people_tracker（lidar:=mid360），发 /guide/people，按高度判断儿童
- M5.3/M5.5 讲解模式可切换（指向展品 / 面向观众）；到站没人先问「大家跟上了吗」，只有一个儿童时用儿童模式，观众走光挥手告别
- 加装水平前置 USB 相机（front_camera），camera_jpeg + vision/watch.py：YOLO 人、YuNet 正脸、MediaPipe 手势
- M5.9 视觉唤醒（正脸 + 雷达距离 3 m 内 + 唤醒词），保留直接唤醒可切换；M5.1 手势代码完成，验收待摄像头实测
- 展品识别（M5.3/M5.4/M5.7/M5.8）取消，原因写入 PLAN
- 同时提交用户的导航改进、Gazebo 性能处理、Isaac 训练脚本和 MuJoCo 策略（demo 视频不入库）

Co-Authored-By: Claude Opus 5.5 <noreply@anthropic.com>

File: ws/src/g1_guide/urdf/g1_glide.urdf (robot description, URDF)
Before this commit: robot g1_29dof_mode_11, 41 links, 40 joints
Links:
- added link front_camera_link
- added link front_camera_optical_frame
Joints:
- added joint front_camera_joint: type fixed, parent torso_link, child front_camera_link, origin xyz=0.09 0.0 0.50 rpy=0 0 0
- added joint front_camera_optical_joint: type fixed, parent front_camera_link, child front_camera_optical_frame, origin xyz=0 0 0 rpy=-1.57079632679 0 -1.57079632679

File: ws/src/g1_guide/urdf/g1_glide_mid360.urdf (robot description, URDF)
Before this commit: robot g1_29dof_mode_11, 41 links, 40 joints
Links:
- added link front_camera_link
- added link front_camera_optical_frame
Joints:
- added joint front_camera_joint: type fixed, parent torso_link, child front_camera_link, origin xyz=0.09 0.0 0.50 rpy=0 0 0
- added joint front_camera_optical_joint: type fixed, parent front_camera_link, child front_camera_optical_frame, origin xyz=0 0 0 rpy=-1.57079632679 0 -1.57079632679
